File: kicad/led-backlight/led-backlight.kicad_pcb (KiCad board)
At the start: 2 copper layers, 63 x 53 mm, 19 parts, among them J1 Conn_01x03, J2 JST_XH_S4B-XH-A_1x04_P2.50mm_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, J3 JST_XH_S4B-XH-A_1x04_P2.50mm_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, J4 JST_XH_S2B-XH-A_1x02_P2.50mm_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, Q1 BSS138, SW1 SW_MEC_5E, U1 AMS1117-3.3, U2 SeeeduinoXIAO, U3 AMS1117-3.3

Commit message: idk can't remember
Parts:
- removed J1: Conn_01x03, Connector_JST:JST_XH_S3B-XH-A_1x03_P2.50mm_Horizontal
- added REF**: jst_xh_conn_1x03_horizontal, initeq:jst_xh_conn_1x03_horizontal, F.Cu at (172.3, 99.5)
- J2, J3: value JST_XH_S4B-XH-A_1x04_P2.50mm_Horizontal -> jst_xh_conn_1x04_horizontal; footprint Connector_JST:JST_XH_S4B-XH-A_1x04_P2.50mm_Horizontal -> initeq:jst_xh_conn_1x04_horizontal
- J4: value JST_XH_S2B-XH-A_1x02_P2.50mm_Horizontal -> jst_xh_conn_1x02_horizontal; footprint Connector_JST:JST_XH_S2B-XH-A_1x02_P2.50mm_Horizontal -> initeq:jst_xh_conn_1x02_horizontal
- RV1: footprint Connector_JST:JST_XH_S3B-XH-A_1x03_P2.50mm_Horizontal -> initeq:jst_xh_conn_1x03_horizontal
- moved J3 3.80 mm to (176.4, 131.2), turned to 180 degrees
- moved J2 3.80 mm to (206.1, 100.1), turned to 0 degrees
- moved RV1 2.50 mm to (202.3, 136.1), turned to 0 degrees
- moved J4 1.28 mm to (202.1, 124.5), turned to 0 degrees
Connections:
- J2 pad 1: GND -> +5V
- J2 pad 2: /mcu_board/mode_btn -> /mcu_board/mode_ref
- J2 pad 3: /mcu_board/mode_ref -> /mcu_board/mode_btn
- J2 pad 4: +5V -> (no net)
- J3 pad 2: /mcu_board/mode_ref -> /mcu_board/mode_btn
- J3 pad 3: /mcu_board/mode_btn -> /mcu_board/mode_ref
Routing:
- net +5V: track 155.2 -> 154.1 mm
